Commit message: fix: core architectural fixes and YOLO integration
- Refined URDF with base_footprint and sensor plugins
- Enhanced Gazebo world with barriers, ramp, and traffic cones
- Implemented real YOLOv8 integration in tabela_detector.py
- Optimized Nav2 inflation radius for tight maneuvers

File: ika_description/urdf/ika.urdf (robot description, URDF)
Before this commit: robot ika, 3 links, 2 joints
Links:
- added link base_footprint
Joints:
- added joint base_joint: type fixed, parent base_footprint, child base_link, origin xyz=0 0 0.36 rpy=0 0 0
- joint camera_joint: origin xyz=0.65 0 0.1 rpy=0 0 0 -> xyz=0.65 0 0.2 rpy=0 0 0
- joint lidar_joint: origin xyz=0.5 0 0.38 rpy=0 0 0 -> xyz=0.5 0 0.385 rpy=0 0 0

Commit message: feat: migrate to ROS 2 Jazzy and Gazebo Sim (Harmonic)
- Updated URDF with gz-sim (Ignition) plugins for diff drive, sensors, and imu
- Refactored launch file to use ros_gz_sim and parameter_bridge
- Established communication bridge between ROS 2 topics and Gazebo Sim

File: ika_description/urdf/ika.urdf (robot description, URDF)
Before this commit: robot ika, 4 links, 3 joints
Links:
- added link rl_wheel, mass 2.5; collision cylinder length=0.08 radius=0.2; visual cylinder length=0.08 radius=0.2
- added link rr_wheel, mass 2.5; collision cylinder length=0.08 radius=0.2; visual cylinder length=0.08 radius=0.2
Joints:
- added joint rl_wheel_joint: type continuous, parent base_link, child rl_wheel, origin xyz=-0.4 0.575 -0.16, axis 0 1 0
- added joint rr_wheel_joint: type continuous, parent base_link, child rr_wheel, origin xyz=-0.4 -0.575 -0.16, axis 0 1 0
- joint camera_joint: origin xyz=0.65 0 0.2 rpy=0 0 0 -> xyz=0.65 0 0.2
- joint lidar_joint: origin xyz=0.5 0 0.385 rpy=0 0 0 -> xyz=0.5 0 0.385
